File: board/gba-dumper.kicad_pcb (KiCad board)
At the start: 2 copper layers, 60 x 60 mm, 2 parts

Commit message: fix: errata board
Routing:
- net Net-(U2-GND): vias 33 -> 36
Other:
- board text added: "GBA Dumper Version 0.1.1 @pakutoma 2025"
- board text removed: "GBA Dumper Version 0.1.0 @pakutoma 2025"
